File: ATtiny3/MosfetDriver.kicad_sch (KiCad schematic)
At the start: 5 parts, among them Q2 SMD-MOSFET-N-CH-20V-2.1A-CJ23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

Commit message: Primo ordine JLCPCB
Parts:
- dq2: renamed from D2; footprint Diode_SMD:D_0805_2012Metric -> Diode_SMD:D_SOD-123; LCSC C84354 -> C8598
- led2: renamed from LED2; value SMD-LED-CLEAR-RED_0805_ -> SMD-LED-CLEAR-0805; footprint Library:LED-0805 -> LED_SMD:LED_0805_2012Metric; LCSC C2764885 -> C2296; MPN 17-215SURC_S530-A2_TR8 -> (none); SKU 304090046 -> (none)
- q2: renamed from Q2; value SMD-MOSFET-N-CH-20V-2.1A-CJ2302_SOT-23_ -> SMD-MOSFET-N-CH; footprint Library:SOT95P240X115-3N -> Package_TO_SOT_SMD:SOT-23; LCSC C91104 -> C20917; MPN CJ2302 -> (none); SKU 305030015 -> (none)
- rgate2: renamed from R2; value SMD-RES-4.7K-5%-1_8W_0805_ -> 10K; footprint Resistor_SMD:R_0815_2038Metric -> Resistor_SMD:R_0805_2012Metric; LCSC C473295 -> C17414
- rled2: renamed from RLED2; LCSC C365277 -> C17557
Other:
- moved on the sheet: dq2, q2, rgate2

Commit message: Primo ordine JLCPCB
Parts:
- dq2: symbol ULN2803-Mosfet-S2-Mini-rescue:SMD-DIODE-SCHOTTKY-20V-1A_SOD-123_-OPL_Discrete -> ULN2803-Mosfet-S2-Mini-rescue:SMD-DIODE-SCHOTTKY-SOD-123; MPN B5819W -> (none); SKU 304020034 -> (none)
- led2: symbol ULN2803-Mosfet-S2-Mini-rescue:SMD-LED-CLEAR-RED_0805_-OPL_Opto -> ULN2803-Mosfet-S2-Mini-rescue:SMD-LED-YELLOW-0805
- q2: symbol ULN2803-Mosfet-S2-Mini-rescue:SMD-MOSFET-N-CH-20V-2.1A-CJ2302_SOT-23_-OPL_Discrete -> ULN2803-Mosfet-S2-Mini-rescue:SMD-MOSFET-N-CH-SOT-23
Changed lines of the file:
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@@
 	)
 	(symbol
-		(lib_id "ULN2803-Mosfet-S2-Mini-rescue:SMD-LED-CLEAR-RED_0805_-OPL_Opto")
+		(lib_id "ULN2803-Mosfet-S2-Mini-rescue:SMD-LED-YELLOW-0805")
 		(at 60.96 48.26 270)
 		(unit 1)
@@
 		)
 		(property "Footprint" "LED_SMD:LED_0805_2012Metric"
-			(at 60.96 48.26 0)
-			(effects
-				(font
-					(size 1.27 1.27)
+			(at 57.912 58.928 0)
+			(effects
+				(font
+					(size 0.762 0.762)
 				)
 				(hide yes)
@@
 		)
 		(property "LCSC" "C2296"
-			(at 60.96 48.26 90)
-			(effects
-				(font
-					(size 1.27 1.27)
-				)
+			(at 54.102 50.038 0)
+			(effects
+				(font
+					(size 0.762 0.762)
+				)
+				(justify left bottom)
 				(hide yes)
 			)
@@
 	)
 	(symbol
-		(lib_id "ULN2803-Mosfet-S2-Mini-rescue:SMD-DIODE-SCHOTTKY-20V-1A_SOD-123_-OPL_Discrete")
+		(lib_id "ULN2803-Mosfet-S2-Mini-rescue:SMD-DIODE-SCHOTTKY-SOD-123")
 		(at 80.01 56.515 90)
 		(unit 1)
@@
 		)
 		(property "Footprint" "Diode_SMD:D_SOD-123"
-			(at 80.01 56.515 0)
-			(effects
-				(font
-					(size 1.27 1.27)
-				)
+			(at 77.216 54.737 0)
+			(effects
+				(font
+					(size 1.27 1.27)
+				)
+				(justify left)
 				(hide yes)
 			)
@@
 			)
 		)
-		(property "MPN" "B5819W"
-			(at 76.2 55.753 0)
-			(effects
-				(font
-					(size 0.508 0.508)
-				)
-				(hide yes)
-			)
-		)
-		(property "SKU" "304020034"
-			(at 76.2 55.753 0)
-			(effects
-				(font
-					(size 0.508 0.508)
-				)
-				(hide yes)
-			)
-		)
 		(property "LCSC" "C8598"
-			(at 80.01 56.515 90)
-			(effects
-				(font
-					(size 1.27 1.27)
-				)
+			(at 84.836 54.737 0)
+			(effects
+				(font
+					(size 0.762 0.762)
+				)
+				(justify left)
 				(hide yes)
 			)
@@
 	)
 	(symbol
-		(lib_id "ULN2803-Mosfet-S2-Mini-rescue:SMD-MOSFET-N-CH-20V-2.1A-CJ2302_SOT-23_-OPL_Discrete")
+		(lib_id "ULN2803-Mosfet-S2-Mini-rescue:SMD-MOSFET-N-CH-SOT-23")
 		(at 73.66 43.18 0)
 		(unit 1)
@@
 		)
 		(property "Footprint" "Package_TO_SOT_SMD:SOT-23"
-			(at 73.66 43.18 0)
-			(effects
-				(font
-					(size 1.27 1.27)
-				)
+			(at 75.184 50.8 0)
+			(effects
+				(font
+					(size 0.762 0.762)
+				)
+				(justify left)
 				(hide yes)
 			)
@@
 			)
 		)
-		(property "Description" ""
-			(at 73.66 43.18 0)
-			(effects
-				(font
-					(size 1.27 1.27)
-				)
+		(property "Description" "https://www.lcsc.com/datasheet/lcsc_datasheet_1811081213_Alpha---Omega-Semicon-AO3400A_C20917.pdf"
+			(at 75.184 47.752 0)
+			(effects
+				(font
+					(size 0.762 0.762)
+				)
+				(justify left)
 				(hide yes)
 			)
@@
 		)
 		(property "LCSC" "C20917"
-			(at 73.66 43.18 0)
-			(effects
-				(font
-					(size 1.27 1.27)
-				)
-				(hide yes)
-			)
+			(at 75.184 49.276 0)
+			(effects
+				(font
+					(size 0.762 0.762)
+				)
+				(justify left)
+				(hide yes)
+			)
